File: PCB/ZeroUNOBridge/ZeroUNOBridge.brd (EAGLE design)
At the start: 30.2 x 62.2 mm, 37 parts, among them J3 RASPBERRYPI-40-PIN-GPIO, Q1 BSS138, Q2 BSS138, Q3 BSS138, Q4 BSS138, Q5 BSS138, Q6 BSS138, U1 ATMEGA328P_PDIP_EZ

Commit message: Final Changes
-DRC clear
-Renumber
Parts:
- removed J4: (no value), SparkFun-Connectors:SCREWTERMINAL-3.5MM-5
- added J2: RASPBERRYPI-40-PIN-GPIO, SparkFun-Boards:2X20-SHROUDED
- J3: value RASPBERRYPI-40-PIN-GPIO -> (none); device SparkFun-Boards:2X20-SHROUDED -> SparkFun-Connectors:SCREWTERMINAL-3.5MM-5
- LED3: value BLUE -> GREEN
- LED4: value GREEN -> BLUE
- R10: value 10K -> PHOTOCELLPTH; device SparkFun-Resistors:0603-RES -> SparkFun-Sensors:PHOTOCELL
- R16: value 10K -> 1M
- R20, R8: value 10K -> 330
- R4, R5: value 330 -> 10K
- R6: value 1M -> 10K
- R7: value PHOTOCELLPTH -> 10K; device SparkFun-Sensors:PHOTOCELL -> SparkFun-Resistors:0603-RES
- moved R20 38.2 mm to (21.6, 10.2), turned to 0 degrees
- moved R4 38.2 mm to (19.1, 48.3), turned to 270 degrees
- moved LED3 33.8 mm to (2.54, 39.4)
- moved LED4 33.8 mm to (21.6, 11.4)
- moved R19 31.8 mm to (21.6, 14.0)
- moved Q6 31.7 mm to (21.6, 16.5)
- moved J3 29.3 mm to (7.62, 3.81)
- moved R6 25.7 mm to (19.1, 41.9), turned to 270 degrees
- moved R5 20.5 mm to (21.6, 45.7)
- moved R7 20.1 mm to (21.6, 39.4), turned to 180 degrees
- moved R10 18.8 mm to (2.54, 33.0)
- moved R16 16.6 mm to (5.08, 20.3), turned to 90 degrees
- moved R12 14.1 mm to (5.33, 32.1)
- moved Q3 12.7 mm to (21.6, 35.6)
- moved R13 9.25 mm to (19.1, 29.2), turned to 270 degrees
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Connections:
- net 3.3V: now also J2.1, J2.17, R14.2, R5.2, R7.2; no longer J3.1, J3.17, R13.2, R15.2, R9.2
- net 5V: now also J2.2, J2.4, R13.2, R15.2, R4.2, R6.2, R9.2; no longer J3.2, J3.4, R10.2, R14.2, R16.2, R20.2, R8.2
- net GND: now also J2.14, J2.20, J2.25, J2.30, J2.34, J2.39, J2.6, J2.9, R10.1; no longer J3.14, J3.20, J3.25, J3.30, J3.34, J3.39, J3.6, J3.9, R7.1
- net MISO_HV: now also Q6.3; no longer Q5.3
- net MISO_LV: now also J2.21, Q6.2, R19.1; no longer J3.21, Q5.2, R17.1
- net MOSI_HV: now also R13.1; no longer R16.1
- net MOSI_LV: now also J2.19, R14.1; no longer J3.19, R15.1
- net N$1: now also J2.37, R20.2; no longer J3.37, R4.2
- net N$5: now also LED4.A, R20.1; no longer LED3.A, R4.1
- net N$6: now also R8.1; no longer R5.1
- net N$7: now also LED3.A, R8.2; no longer LED4.A, R5.2
- net N$9: now also R10.2, R12.1; no longer R7.2, R8.1
- net PIN10~: now also J3.5; no longer J4.5
- net PIN3~: now also J3.1; no longer J4.1
- net PIN5~: now also J3.2; no longer J4.2
- net PIN6~: now also J3.3; no longer J4.3
- net PIN9~: now also J3.4; no longer J4.4
- net RESET_HV: now also Q1.3, R4.1; no longer Q6.3, R20.1
- net RESET_LV: now also J2.22, Q1.2, R5.1; no longer J3.22, Q6.2, R19.1
- net RX_HV: now also Q2.3, R6.1; no longer Q1.3, R10.1
- net RX_LV: now also J2.10, Q3.2; no longer J3.10, Q2.2
- net SCLK_HV: now also Q5.3, R15.1; no longer Q3.3, R14.1
- net SCLK_LV: now also J2.23, Q5.2, R17.1; no longer J3.23, Q3.2, R13.1
- net TX_HV: now also Q3.3, R9.1; no longer Q2.3, R12.1
- net TX_LV: now also J2.8, Q2.2, R7.1; no longer J3.8, Q1.2, R9.1
- net XTAL1: now also R16.2; no longer R6.2
- net XTAL2: now also R16.1; no longer R6.1
